File: 17_CAN_Controller.kicad_pcb (KiCad board)
At the start: 2 copper layers, 20.3 x 20.3 mm, 15 parts, among them J1 Conn_01x01, J2 Conn_01x01, J3 Conn_01x01, J5 Conn_01x01, J6 Conn_01x01, J7 Conn_01x01, J8 Conn_01x01, J9 Conn_01x01, U1 MCP2515-xSO, Y1 X322516MLB4SI

Commit message: maj split librairies
Parts:
- J1, J2, J3, J5, J6, J7, J8, J9: footprint Chimere:Castellated_conn -> Chimere_mods:Castellated_conn

Commit message: maj kicad 6
+ correction chemin

+ step
Other:
- net class Default removed
- net class demi-gros removed
- net class gros removed

Commit message: maj réduction de taille
Parts:
- removed J3, J5, J6, J7, J8, J9: Conn_01x01, Chimere_mods:Castellated_conn
- J1: value Conn_01x01 -> Conn_01x08; footprint Chimere_mods:Castellated_conn -> Connector_PinHeader_2.54mm:PinHeader_1x08_P2.54mm_Vertical; moved to B.Cu
- J2: footprint Chimere_mods:Castellated_conn -> Connector_PinHeader_2.54mm:PinHeader_1x01_P2.54mm_Vertical; moved to B.Cu
- moved J2 19.8 mm to (119.4, 81.3)
- moved J1 2.54 mm to (104.1, 63.5)
Connections:
- J1 pad 1: CAN_TX -> 5V
- J2 pad 1: CAN_RX -> GND
- U1 pad 10: Net-(U1-Pad10) -> unconnected-(U1-Pad10)
- U1 pad 11: Net-(U1-Pad11) -> unconnected-(U1-Pad11)
- U1 pad 12: Net-(U1-Pad12) -> unconnected-(U1-Pad12)
- U1 pad 3: Net-(U1-Pad3) -> unconnected-(U1-Pad3)
- U1 pad 4: Net-(U1-Pad4) -> unconnected-(U1-Pad4)
- U1 pad 5: Net-(U1-Pad5) -> unconnected-(U1-Pad5)
- U1 pad 6: Net-(U1-Pad6) -> unconnected-(U1-Pad6)
Other:
- board size 20.3 x 20.3 mm -> 17.8 x 20.3 mm
- board text added: "17_CAN_Controller"
- board text added: "2022/11/03"
- board text removed: "2021/06/01"
- board text removed: "github.com/ ThierryOrlandi/ 17_CAN_Controller"
